File: hardware/i2s-muliplexer/i2s-multiplexer/i2s-multiplexer.kicad_pcb (KiCad board)
At the start: 2 copper layers, 18 parts, among them J1 Conn_01x07, J10 Conn_01x04, J2 Conn_01x04, J3 Conn_01x04, J4 Conn_01x04, J5 Conn_01x04, J6 Conn_01x04, J7 Conn_01x04, J8 Conn_01x04, J9 Conn_01x04, U1 74HC4051, U2 74HC4051, U3 74HC4051, U4 74HC4051, U5 74HC126

Commit message: Using buffers
Parts:
- removed J1: Conn_01x07, Connector_PinHeader_2.54mm:PinHeader_1x07_P2.54mm_Vertical
- removed J10, J2, J3, J4, J5, J6, J7, J8, J9: Conn_01x04, Connector_PinHeader_2.54mm:PinHeader_1x04_P2.54mm_Vertical
- removed R1, R2, R3: 10K, Resistor_SMD:R_0805_2012Metric_Pad1.15x1.40mm_HandSolder
- removed U1, U2, U3, U4: 74HC4051, Package_SO:SOIC-16_3.9x9.9mm_P1.27mm
- removed U5: 74HC126, Package_SO:SOIC-14_3.9x8.7mm_P1.27mm
Routing:
- net +3V3: track 89.1 -> 0.00 mm

Commit message: Initial PCB design
Parts:
- added J1: Conn_01x05, Connector_PinHeader_2.54mm:PinHeader_1x05_P2.54mm_Vertical, F.Cu at (57.9, 38.6)
- added J2: Conn_01x05, Connector_PinHeader_2.54mm:PinHeader_1x05_P2.54mm_Vertical, F.Cu at (40.4, 38.6)
- added J3: Conn_01x05, Connector_PinHeader_2.54mm:PinHeader_1x05_P2.54mm_Vertical, F.Cu at (75.7, 38.6)
- added J4: Conn_01x05, Connector_PinHeader_2.54mm:PinHeader_1x05_P2.54mm_Vertical, F.Cu at (46.2, 75.9)
- added J5: Conn_01x05, Connector_PinHeader_2.54mm:PinHeader_1x05_P2.54mm_Vertical, F.Cu at (29.7, 75.9)
- added J6: Conn_01x07, Connector_PinHeader_2.54mm:PinHeader_1x07_P2.54mm_Vertical, F.Cu at (67.8, 75.9)
- added J7: Conn_01x05, Connector_PinHeader_2.54mm:PinHeader_1x05_P2.54mm_Vertical, F.Cu at (94.5, 60.2)
- added R1: 10K, Resistor_SMD:R_0805_2012Metric_Pad1.15x1.40mm_HandSolder, F.Cu at (77.5, 45.2)
- added R2: 10K, Resistor_SMD:R_0805_2012Metric_Pad1.15x1.40mm_HandSolder, F.Cu at (82.0, 45.2)
- added R3: 10K, Resistor_SMD:R_0805_2012Metric_Pad1.15x1.40mm_HandSolder, F.Cu at (79.8, 45.2)
- added R4: 10K, Resistor_SMD:R_0805_2012Metric_Pad1.15x1.40mm_HandSolder, F.Cu at (84.3, 45.2)
- added R5: 10K, Resistor_SMD:R_0805_2012Metric_Pad1.15x1.40mm_HandSolder, F.Cu at (87.6, 45.2)
- added R6: 10K, Resistor_SMD:R_0805_2012Metric_Pad1.15x1.40mm_HandSolder, F.Cu at (66.0, 70.9)
- added REF**: MountingHole_3.2mm_M3_ISO7380, MountingHole:MountingHole_3.2mm_M3_ISO7380, F.Cu at (96.5, 35.6)
- added REF**: MountingHole_3.2mm_M3_ISO7380, MountingHole:MountingHole_3.2mm_M3_ISO7380, F.Cu at (24.6, 35.6)
- added REF**: MountingHole_3.2mm_M3_ISO7380, MountingHole:MountingHole_3.2mm_M3_ISO7380, F.Cu at (24.1, 79.8)
- added REF**: MountingHole_3.2mm_M3_ISO7380, MountingHole:MountingHole_3.2mm_M3_ISO7380, F.Cu at (96.3, 80.0)
- added U1: 74HC126, Package_SO:SOIC-14_3.9x8.7mm_P1.27mm, F.Cu at (69.3, 46.2)
- added U2: 74HC126, Package_SO:SOIC-14_3.9x8.7mm_P1.27mm, F.Cu at (51.6, 46.2)
- added U3: 74HC126, Package_SO:SOIC-14_3.9x8.7mm_P1.27mm, F.Cu at (34.1, 46.2)
- added U4: 74HC126, Package_SO:SOIC-14_3.9x8.7mm_P1.27mm, F.Cu at (36.0, 68.3)
- added U5: 74HC126, Package_SO:SOIC-14_3.9x8.7mm_P1.27mm, F.Cu at (52.4, 68.3)
- added U6: 74HC126, Package_SO:SOIC-14_3.9x8.7mm_P1.27mm, F.Cu at (84.8, 54.6)
- added U7: 74LS138, Package_SO:SOIC-16_3.9x9.9mm_P1.27mm, F.Cu at (74.9, 68.3)
Routing:
- net /LRCLK: track 0.00 -> 149.0 mm, vias 0 -> 8
- net /MCLK: track 0.00 -> 122.5 mm, vias 0 -> 6
- net /BCLK: track 0.00 -> 120.3 mm, vias 0 -> 14
- net /DATA: track 0.00 -> 95.4 mm, vias 0 -> 12
- net /CH_EN_2: track 0.00 -> 93.1 mm, vias 0 -> 6
- net /CH_EN_3: track 0.00 -> 86.5 mm, vias 0 -> 7
- net /CH_EN_1: track 0.00 -> 86.4 mm, vias 0 -> 7
- net /CH_EN_0: track 0.00 -> 64.4 mm, vias 0 -> 7
- net /CH_EN_4: track 0.00 -> 57.6 mm, vias 0 -> 7
- net /MCLK_EN: track 0.00 -> 39.8 mm, vias 0 -> 4
- net Net-(R5-Pad2): track 0.00 -> 21.4 mm, vias 0 -> 2
- net /S0: track 0.00 -> 21.4 mm, vias 0 -> 1
- net /DATA_OUT: track 0.00 -> 21.1 mm, vias 0 -> 2
- net GND: track 0.00 -> 20.4 mm, vias 0 -> 12
- net /S1: track 0.00 -> 16.1 mm, vias 0 -> 1
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- added copper zone on F.Cu, net +3V3
- added copper zone on B.Cu, net GND
Other:
- board outline added: 81 x 53.6 mm
- board text added: "+3.3V"
- board text added: "ADDR"
- board text added: "BCLK"
- board text added: "DATA"
- board text added: "GND"
- board text added: "I2S OUT"
- board text added: "I2S Source 0"
- board text added: "I2S Source 1"
- board text added: "I2S Source 2"
- board text added: "I2S Source 3"
- board text added: "I2S Source 4"
- board text added: "LRCLK"
- board text added: "MCLK"
- board text added: "MCLK_EN"
- board text added: "S0"
- board text added: "S1"
- board text added: "S2"
- board text added: "SRC_EN"
