File: hardware/power-board/power-board.kicad_sch (KiCad schematic)
At the start: 9 parts, among them J1 Screw_Terminal_01x02, J2 Screw_Terminal_01x08, J3 Screw_Terminal_01x08, U1 TSR_1-2433, U2 TSR_1-2450

Commit message: Updated explanatory notes on schematic
Other:
- note added: "As inside only need low luminosity => low current >= 1mA R = 3.3V - 2V / 1mA = 1 300 Ohm => 1K Ohm"
- note added: "As inside only need low luminosity => low current >= 1mA R = 5V - 3.3V / 1mA = 1 700 Ohm => 1K Ohm"
- note removed: "As inside only need low current >= 1mA R = 3.3V - 2V / 1mA = 1 300 Ohm => 1K Ohm"
- note removed: "As inside only need low current >= 1mA R = 5V - 3.3V / 1mA = 1 700 Ohm => 1K Ohm"
Changed lines of the file:
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@@
     (effects (font (size 1.27 1.27)) (justify left bottom))
   )
-  (text "As inside only need low current  >= 1mA\nR = 3.3V - 2V / 1mA = 1 300 Ohm => 1K Ohm\n\n"
-    (at 100.33 90.17 0)
+  (text "As inside only need low luminosity => low current  >= 1mA\nR = 3.3V - 2V / 1mA = 1 300 Ohm => 1K Ohm\n\n"
+    (at 96.52 90.17 0)
     (effects (font (size 1.27 1.27)) (justify left bottom))
   )
@@
   )
   (text "A red LED typically drops around 1.7 to 2.0 volts.\n"
-    (at 100.33 83.82 0)
+    (at 96.52 83.82 0)
     (effects (font (size 1.27 1.27)) (justify left bottom))
   )
@@
     (effects (font (size 1.27 1.27) (thickness 0.254) bold) (justify right bottom))
   )
-  (text "As inside only need low current >= 1mA\nR = 5V - 3.3V / 1mA = 1 700 Ohm => 1K Ohm\n\n"
-    (at 101.6 147.32 0)
+  (text "As inside only need low luminosity => low current >= 1mA\nR = 5V - 3.3V / 1mA = 1 700 Ohm => 1K Ohm\n\n"
+    (at 96.52 147.32 0)
     (effects (font (size 1.27 1.27)) (justify left bottom))
   )
-  (text "A blue LED may drop around 3 to 3.3 volts." (at 101.6 140.97 0)
+  (text "A blue LED may drop around 3 to 3.3 volts." (at 96.52 140.97 0)
     (effects (font (size 1.27 1.27)) (justify left bottom))
   )
