File: hardware/select-buttons-board/select-buttons-board/select-buttons-board.kicad_sch (KiCad schematic)
At the start: 10 parts, among them SW1 A, SW2 B, SW3 C, SW4 D, U1 MCP23017_SO

Commit message: Initial schematic of select-button-board
Parts:
- added J1: conn_br, Connector_JST:JST_PH_B5B-PH-K_1x05_P2.00mm_Vertical, symbol Connector_Generic:Conn_01x05
- added JP1, JP2, JP3: SolderJumper_2_Open, symbol Jumper:SolderJumper_2_Open
- added R1, R2, R3: 10k, symbol Device:R_Small
- renumbered R1 to R4, R2 to R5, R3 to R6, R4 to R7, R5 to R8
Connections:
- net +3V3: now also J1.2 (Pin_2), JP1.2 (B), JP2.2 (B), JP3.2 (B)
- net GND: now also J1.1 (Pin_1), R1.2, R2.2, R3.2
- net SCK: now reaches U1.12 (SCK)
- net SDA: now reaches U1.13 (SDA)
- net SDA: now also J1.3 (Pin_3)
- net at U1.15 (A0): now also JP1.1 (A), R1.1
- net at U1.16 (A1): now also JP2.1 (A), R2.1
- net at U1.17 (A2): now also JP3.1 (A), R3.1
- net ~{INT}: now reaches U1.20 (INTA)
- net ~{INT}: now also J1.5 (Pin_5)
- new net SCL: J1.4 (Pin_4)
- no-connect marks 0 -> 13
Other:
- note added: "Address selection"
- note added: "MCP23017 is set up by software as follows: All pins: input Interrupts mirroring: false, open_drain: false, polarity: Low interrupt-on-pin change: rising"
- note removed: "INCOMPLETE"
- moved on the sheet: R4
