File: hardware/select-buttons-board/select-buttons-board.kicad_sch (KiCad schematic)
At the start: 17 parts, among them J1 conn_br, SW1 A, SW2 B, SW3 C, SW4 D, U1 MCP23017_SO

Commit message: Corrections as of now
Connections:
- net SCL is gone; now on net SCK: J1.4 (Pin_4)
- net ~{INT} renamed ~{INTR}
Other:
- note added: "JP3 (A2) JP2 (A1) JP1 (A0) I2C Address O O O 0x20 O O C 0x21 O C O 0x22 O C C 0x23 C O O 0x24 C O C 0x25 C C O 0x26 C C C 0x27"
- note added: "Jumpers and I2C address"
- note added: "O = OPEN, C = CLOSED"
Changed lines of the file:
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@@
     (stroke (width 0) (type default) (color 0 0 0 0))
   )
-  (wire (pts (xy 109.22 143.51) (xy 130.81 143.51))
+  (wire (pts (xy 118.11 143.51) (xy 130.81 143.51))
     (stroke (width 0) (type default) (color 0 0 0 0))
   )
@@
     (stroke (width 0) (type default) (color 0 0 0 0))
   )
+  (polyline (pts (xy 40.64 139.7) (xy 40.64 161.29))
+    (stroke (width 0) (type default) (color 0 0 0 0))
+  )
   (wire (pts (xy 170.18 87.63) (xy 170.18 96.52))
     (stroke (width 0) (type default) (color 0 0 0 0))
   )
-  (wire (pts (xy 99.06 80.01) (xy 107.95 80.01))
+  (wire (pts (xy 105.41 80.01) (xy 107.95 80.01))
     (stroke (width 0) (type default) (color 0 0 0 0))
   )
@@
     (stroke (width 0) (type default) (color 0 0 0 0))
   )
+  (polyline (pts (xy 24.13 132.08) (xy 24.13 133.35))
+    (stroke (width 0) (type default) (color 0 0 0 0))
+  )
+  (polyline (pts (xy 92.71 168.91) (xy 92.71 132.08))
+    (stroke (width 0) (type default) (color 0 0 0 0))
+  )
+  (polyline (pts (xy 24.13 168.91) (xy 92.71 168.91))
+    (stroke (width 0) (type default) (color 0 0 0 0))
+  )
   (wire (pts (xy 185.42 90.17) (xy 185.42 96.52))
     (stroke (width 0) (type default) (color 0 0 0 0))
@@
     (stroke (width 0) (type default) (color 0 0 0 0))
   )
-  (wire (pts (xy 99.06 64.77) (xy 107.95 64.77))
+  (polyline (pts (xy 24.13 133.35) (xy 24.13 168.91))
+    (stroke (width 0) (type default) (color 0 0 0 0))
+  )
+  (polyline (pts (xy 27.94 139.7) (xy 27.94 161.29))
+    (stroke (width 0) (type default) (color 0 0 0 0))
+  )
+  (polyline (pts (xy 27.94 143.51) (xy 88.9 143.51))
+    (stroke (width 0) (type default) (color 0 0 0 0))
+  )
+  (wire (pts (xy 105.41 64.77) (xy 107.95 64.77))
     (stroke (width 0) (type default) (color 0 0 0 0))
   )
@@
     (stroke (width 0) (type default) (color 0 0 0 0))
   )
+  (polyline (pts (xy 88.9 161.29) (xy 88.9 139.7))
+    (stroke (width 0) (type default) (color 0 0 0 0))
+  )
   (wire (pts (xy 74.93 100.33) (xy 74.93 109.22))
     (stroke (width 0) (type default) (color 0 0 0 0))
@@
     (stroke (width 0) (type default) (color 0 0 0 0))
   )
-  (wire (pts (xy 109.22 146.05) (xy 130.81 146.05))
+  (wire (pts (xy 118.11 146.05) (xy 130.81 146.05))
+    (stroke (width 0) (type default) (color 0 0 0 0))
+  )
+  (polyline (pts (xy 57.15 161.29) (xy 55.88 161.29))
     (stroke (width 0) (type default) (color 0 0 0 0))
   )
@@
     (stroke (width 0) (type default) (color 0 0 0 0))
   )
+  (polyline (pts (xy 27.94 139.7) (xy 27.94 143.51))
+    (stroke (width 0) (type default) (color 0 0 0 0))
+  )
+  (polyline (pts (xy 57.15 139.7) (xy 57.15 161.29))
+    (stroke (width 0) (type default) (color 0 0 0 0))
+  )
   (wire (pts (xy 185.42 90.17) (xy 185.42 85.09))
     (stroke (width 0) (type default) (color 0 0 0 0))
@@
     (stroke (width 0) (type default) (color 0 0 0 0))
   )
-  (wire (pts (xy 99.06 62.23) (xy 107.95 62.23))
+  (wire (pts (xy 105.41 62.23) (xy 107.95 62.23))
     (stroke (width 0) (type default) (color 0 0 0 0))
   )
@@
     (stroke (width 0) (type default) (color 0 0 0 0))
   )
+  (polyline (pts (xy 27.94 161.29) (xy 88.9 161.29))
+    (stroke (width 0) (type default) (color 0 0 0 0))
+  )
+  (polyline (pts (xy 88.9 139.7) (xy 27.94 139.7))
+    (stroke (width 0) (type default) (color 0 0 0 0))
+  )
+  (polyline (pts (xy 72.39 139.7) (xy 72.39 161.29))
+    (stroke (width 0) (type default) (color 0 0 0 0))
+  )
   (wire (pts (xy 200.66 92.71) (xy 200.66 85.09))
     (stroke (width 0) (type default) (color 0 0 0 0))
@@
     (stroke (width 0) (type default) (color 0 0 0 0))
   )
-  (wire (pts (xy 109.22 148.59) (xy 130.81 148.59))
+  (wire (pts (xy 118.11 148.59) (xy 130.81 148.59))
     (stroke (width 0) (type default) (color 0 0 0 0))
   )
@@
     (stroke (width 0) (type default) (color 0 0 0 0))
   )
+  (polyline (pts (xy 92.71 132.08) (xy 24.13 132.08))
+    (stroke (width 0) (type default) (color 0 0 0 0))
+  )
   (wire (pts (xy 68.58 102.87) (xy 107.95 102.87))
     (stroke (width 0) (type default) (color 0 0 0 0))
+  )
+  (text "Jumpers and I2C address" (at 29.21 135.89 0)
+    (effects (font (size 1.27 1.27) (thickness 0.254) bold) (justify left bottom))
+  )
+  (text "O = OPEN, C = CLOSED" (at 29.21 167.64 0)
+    (effects (font (size 1.27 1.27)) (justify left bottom))
   )
   (text "Note: Baising the ~{RESET} pin \nis important\nfor the correct operation"
@@
     (effects (font (size 1.27 1.27)) (justify left bottom))
   )
-  (label "SDA" (at 101.6 62.23 0)
-    (effects (font (size 1.27 1.27)) (justify left bottom))
-  )
-  (label "~{INT}" (at 109.22 143.51 0)
-    (effects (font (size 1.27 1.27)) (justify left bottom))
-  )
-  (label "SCL" (at 109.22 146.05 0)
-    (effects (font (size 1.27 1.27)) (justify left bottom))
-  )
-  (label "SDA" (at 109.22 148.59 0)
-    (effects (font (size 1.27 1.27)) (justify left bottom))
-  )
-  (label "~{INT}" (at 101.6 80.01 0)
-    (effects (font (size 1.27 1.27)) (justify left bottom))
-  )
-  (label "SCK" (at 101.6 64.77 0)
-    (effects (font (size 1.27 1.27)) (justify left bottom))
+  (text "JP3 (A2)	JP2 (A1)	JP1 (A0)	I2C Address\n\nO			O			O			0x20\nO			O			C			0x21\nO			C			O			0x22\nO			C			C			0x23\nC			O			O			0x24\nC			O			C			0x25\nC			C			O			0x26\nC			C			C			0x27\n\n"
+    (at 29.21 162.56 0)
+    (effects (font (size 1.27 1.27)) (justify left bottom))
+  )
+  (global_label "SDA" (shape input) (at 105.41 62.23 180) (fields_autoplaced)
+    (effects (font (size 1.27 1.27)) (justify right))
+    (property "Intersheet References" "${INTERSHEET_REFS}" (id 0) (at 99.4288 62.3094 0)
+      (effects (font (size 1.27 1.27)) (justify right) hide)
+    )
+  )
+  (global_label "SDA" (shape input) (at 118.11 148.59 180) (fields_autoplaced)
+    (effects (font (size 1.27 1.27)) (justify right))
+    (property "Intersheet References" "${INTERSHEET_REFS}" (id 0) (at 112.1288 148.5106 0)
+      (effects (font (size 1.27 1.27)) (justify right) hide)
+    )
+  )
+  (global_label "SCK" (shape input) (at 105.41 64.77 180) (fields_autoplaced)
+    (effects (font (size 1.27 1.27)) (justify right))
+    (property "Intersheet References" "${INTERSHEET_REFS}" (id 0) (at 99.2474 64.6906 0)
+      (effects (font (size 1.27 1.27)) (justify right) hide)
+    )
+  )
+  (global_label "SCK" (shape input) (at 118.11 146.05 180) (fields_autoplaced)
+    (effects (font (size 1.27 1.27)) (justify right))
+    (property "Intersheet References" "${INTERSHEET_REFS}" (id 0) (at 111.9474 145.9706 0)
+      (effects (font (size 1.27 1.27)) (justify right) hide)
+    )
+  )
+  (global_label "~{INTR}" (shape input) (at 105.41 80.01 180) (fields_autoplaced)
+    (effects (font (size 1.27 1.27)) (justify right))
+    (property "Intersheet References" "${INTERSHEET_REFS}" (id 0) (at 98.824 79.9306 0)
+      (effects (font (size 1.27 1.27)) (justify right) hide)
+    )
+  )
+  (global_label "~{INTR}" (shape input) (at 118.11 143.51 180) (fields_autoplaced)
+    (effects (font (size 1.27 1.27)) (justify right))
+    (property "Intersheet References" "${INTERSHEET_REFS}" (id 0) (at 111.524 143.4306 0)
+      (effects (font (size 1.27 1.27)) (justify right) hide)
+    )
   )
   (symbol (lib_id "Device:R_Small") (at 68.58 111.76 0) (unit 1)
