File: hardware/source-display-processor/source-display-processor.kicad_sch (KiCad schematic)
At the start: 23 parts, among them J1 conn_br, SW1 SW_Push, U1 MCP23017_SO

Commit message: Changed name of the interrupt to SOURCE_CHANGED
Connections:
- net ~{INTR} renamed ~{SOURCE_CHANGED}
Other:
- note added: "Pulses LOW when the button is pressed and released."
- moved on the sheet: JP1, JP2, JP3, R1, R2, R3, R4

Commit message: Noted that simpler NOT to use interrupt pins
Other:
- note added: "Connecting ~{SOURCE_CHANGED} directly to the button works just as well. Why bother with the INTB pin?"
Changed lines of the file:
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@@
+    (stroke (width 0) (type default) (color 0 0 0 0))
+  )
+  (polyline (pts (xy 85.09 121.92) (xy 137.16 121.92))
     (stroke (width 0) (type default) (color 0 0 0 0))
   )
@@
     (stroke (width 0) (type default) (color 0 0 0 0))
   )
+  (polyline (pts (xy 85.09 114.3) (xy 85.09 121.92))
+    (stroke (width 0) (type default) (color 0 0 0 0))
+  )
   (polyline (pts (xy 110.49 144.78) (xy 49.53 144.78))
     (stroke (width 0) (type default) (color 0 0 0 0))
@@
     (stroke (width 0) (type default) (color 0 0 0 0))
   )
+  (polyline (pts (xy 114.3 85.09) (xy 114.3 114.3))
+    (stroke (width 0) (type default) (color 0 0 0 0))
+  )
   (polyline (pts (xy 45.72 173.99) (xy 114.3 173.99))
     (stroke (width 0) (type default) (color 0 0 0 0))
@@
     (stroke (width 0) (type default) (color 0 0 0 0))
   )
+  (polyline (pts (xy 137.16 121.92) (xy 137.16 114.3))
+    (stroke (width 0) (type default) (color 0 0 0 0))
+  )
   (wire (pts (xy 152.4 156.21) (xy 151.13 156.21))
     (stroke (width 0) (type default) (color 0 0 0 0))
@@
     (stroke (width 0) (type default) (color 0 0 0 0))
   )
+  (polyline (pts (xy 85.09 114.3) (xy 137.16 114.3))
+    (stroke (width 0) (type default) (color 0 0 0 0))
+  )
   (polyline (pts (xy 73.66 27.94) (xy 125.73 27.94))
     (stroke (width 0) (type default) (color 0 0 0 0))
@@
   )
   (polyline (pts (xy 204.47 77.47) (xy 226.06 77.47))
+    (stroke (width 0) (type default) (color 0 0 0 0))
+  )
+  (polyline (pts (xy 124.46 121.92) (xy 124.46 146.05))
     (stroke (width 0) (type default) (color 0 0 0 0))
   )
@@
     (effects (font (size 1.27 1.27)) (justify left bottom))
   )
+  (text "Connecting ~{SOURCE_CHANGED} directly to the button\nworks just as well. Why bother with the INTB pin?"
+    (at 86.36 120.65 0)
+    (effects (font (size 1.27 1.27) (thickness 0.254) bold) (justify left bottom))
+  )
   (text "MCP23017 is set up by software as follows:\nAll pins: input\nInterrupts\n    mirroring: false,\n    open_drain: false,\n    polarity: Low\n    interrupt-on-pin change: descending"

Commit message: CHANGE_SOURCE directly driven from push button
Connections:
- net ~{CHANGE_SOURCE}: now reaches R5.2, SW1.2
- net ~{CHANGE_SOURCE}: now also J1.5 (Pin_5); no longer U1.1 (GPB0)
- net ~{SOURCE_CHANGED}: no longer names the net of U1.19 (INTB)
- net ~{SOURCE_CHANGED}: no longer J1.5 (Pin_5)
Other:
- note removed: "Connecting ~{SOURCE_CHANGED} directly to the button works just as well. Why bother with the INTB pin?"
- note removed: "MCP23017 is set up by software as follows: All pins: input Interrupts mirroring: false, open_drain: false, polarity: Low interrupt-on-pin change: descending"
- note removed: "Pulses LOW when the button is pressed and released."
- moved on the sheet: R5, SW1
